File: electronics/PCB_BQ76925_ATMEGA328P_6S_20A_BMS/Atmega328P.kicad_sch (KiCad schematic)
At the start: 17 parts, among them J5 Conn_01x04, J6 Conn_02x03, U3 ATmega328P-A, U4 AMS1117-5.0, Y1 16Mhz

Commit message: common footprints assigned to symbols
Parts:
- C20, C26, C28: value 10uF -> 10uF/16V; footprint (none) -> Capacitor_SMD:C_0603_1608Metric_Pad1.08x0.95mm_HandSolder
- C21, C22, C25, C27: value 0.1uF -> 100nF/50V; footprint Capacitor_SMD:C_0603_1608Metric_Pad1.08x0.95mm_HandSolder -> Capacitor_SMD:C_0805_2012Metric_Pad1.18x1.45mm_HandSolder
- D6: footprint (none) -> Resistor_SMD:R_0805_2012Metric_Pad1.20x1.40mm_HandSolder
Changed lines of the file:
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@@
 			)
 		)
-		(property "Value" "0.1uF"
+		(property "Value" "100nF/50V"
 			(at 259.08 132.0862 0)
 			(effects
@@
 			)
 		)
-		(property "Footprint" "Capacitor_SMD:C_0603_1608Metric_Pad1.08x0.95mm_HandSolder"
+		(property "Footprint" "Capacitor_SMD:C_0805_2012Metric_Pad1.18x1.45mm_HandSolder"
 			(at 256.54 130.81 0)
 			(effects
@@
 			)
 		)
-		(property "Value" "0.1uF"
+		(property "Value" "100nF/50V"
 			(at 88.9 177.8062 0)
 			(effects
@@
 			)
 		)
-		(property "Footprint" "Capacitor_SMD:C_0603_1608Metric_Pad1.08x0.95mm_HandSolder"
+		(property "Footprint" "Capacitor_SMD:C_0805_2012Metric_Pad1.18x1.45mm_HandSolder"
 			(at 86.36 176.53 0)
 			(effects
@@
 			)
 		)
-		(property "Value" "10uF"
+		(property "Value" "10uF/16V"
 			(at 77.47 177.8062 0)
 			(effects
@@
 			)
 		)
-		(property "Footprint" ""
+		(property "Footprint" "Capacitor_SMD:C_0603_1608Metric_Pad1.08x0.95mm_HandSolder"
 			(at 74.93 176.53 0)
 			(effects
@@
 			)
 		)
-		(property "Value" "0.1uF"
+		(property "Value" "100nF/50V"
 			(at 83.82 45.7262 0)
 			(effects
@@
 			)
 		)
-		(property "Footprint" "Capacitor_SMD:C_0603_1608Metric_Pad1.08x0.95mm_HandSolder"
+		(property "Footprint" "Capacitor_SMD:C_0805_2012Metric_Pad1.18x1.45mm_HandSolder"
 			(at 81.28 44.45 0)
 			(effects
@@
 			)
 		)
-		(property "Value" "10uF"
+		(property "Value" "10uF/16V"
 			(at 72.39 45.2881 0)
 			(effects
@@
 			)
 		)
-		(property "Footprint" ""
+		(property "Footprint" "Capacitor_SMD:C_0603_1608Metric_Pad1.08x0.95mm_HandSolder"
 			(at 69.85 44.45 0)
 			(effects
@@
 			)
 		)
-		(property "Value" "10uF"
+		(property "Value" "10uF/16V"
 			(at 116.84 177.8062 0)
 			(effects
@@
 			)
 		)
-		(property "Footprint" ""
+		(property "Footprint" "Capacitor_SMD:C_0603_1608Metric_Pad1.08x0.95mm_HandSolder"
 			(at 114.3 176.53 0)
 			(effects
@@
 			)
 		)
-		(property "Footprint" ""
+		(property "Footprint" "Resistor_SMD:R_0805_2012Metric_Pad1.20x1.40mm_HandSolder"
 			(at 260.35 74.93 90)
 			(effects
@@
 			)
 		)
-		(property "Value" "0.1uF"
+		(property "Value" "100nF/50V"
 			(at 102.87 45.7262 0)
 			(effects
@@
 			)
 		)
-		(property "Footprint" "Capacitor_SMD:C_0603_1608Metric_Pad1.08x0.95mm_HandSolder"
+		(property "Footprint" "Capacitor_SMD:C_0805_2012Metric_Pad1.18x1.45mm_HandSolder"
 			(at 100.33 44.45 0)
 			(effects

Commit message: schematic components footprint updated
Parts:
- C23, C24: footprint (none) -> Capacitor_SMD:C_0603_1608Metric_Pad1.08x0.95mm_HandSolder
- D7: renamed from D6; symbol Device:LED_Small_Filled -> BQ76925_ATMEGA328P_6S_20A_BMS:LED_Small_Filled
- J5: footprint (none) -> Connector_PinHeader_2.54mm:PinHeader_1x04_P2.54mm_Vertical
- J6: footprint (none) -> Connector_PinHeader_2.54mm:PinHeader_2x03_P2.54mm_Vertical
- Y1: footprint (none) -> Crystal:Crystal_HC49-4H_Vertical
- renumbered C27 to C26, C28 to C27, C26 to C28, R28 to R27, R26 to R28
Other:
- moved on the sheet: C26, C28

Commit message: MCU - Crystal replaced with resonator
Parts:
- removed C23, C24: 22pF, Capacitor_SMD:C_0603_1608Metric_Pad1.08x0.95mm_HandSolder, symbol BQ76925_ATMEGA328P_6S_20A_BMS:C_Small
- removed Y1: 16Mhz, Crystal:Crystal_HC49-4H_Vertical, symbol BQ76925_ATMEGA328P_6S_20A_BMS:Crystal_Small
- added Y2: 16Mhz, Crystal:Resonator_SMD_Murata_CSTxExxV-3Pin_3.0x1.1mm_HandSoldering, symbol BQ76925_ATMEGA328P_6S_20A_BMS:Crystal_GND3_Small
Connections:
- net GND: now also Y2.3
- net XTAL1: now also Y2.1
- net XTAL2: now also Y2.2
Other:
- note added: "MCU - Resonator"
- note removed: "MCU - Crystal"

Commit message: pcb design half complete
Parts:
- renumbered C28 to C21, C20 to C22, C26 to C23, C21 to C24, C22 to C25, C27 to C26, C25 to C27, J6 to J5, J5 to J6, R28 to R27, R27 to R28, Y2 to Y1
Changed lines of the file:
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@@
 		(dnp no)
 		(fields_autoplaced yes)
-		(property "Reference" "#PWR034"
+		(property "Reference" "#PWR031"
 			(at 91.44 138.43 0)
 			(effects
@@
 			(project "BQ76925_ATMEGA328P_6S_20A_BMS"
 				(path "/624a087f-322b-4a70-8c29-0e4f8f018e16/e88de734-726e-4991-811a-b88126c63525"
-					(reference "#PWR034")
+					(reference "#PWR031")
 					(unit 1)
 				)
@@
 		(dnp no)
 		(fields_autoplaced yes)
-		(property "Reference" "C25"
+		(property "Reference" "C27"
 			(at 259.08 129.5462 0)
 			(effects
@@
 			(project "BQ76925_ATMEGA328P_6S_20A_BMS"
 				(path "/624a087f-322b-4a70-8c29-0e4f8f018e16/e88de734-726e-4991-811a-b88126c63525"
-					(reference "C25")
+					(reference "C27")
 					(unit 1)
 				)
@@
 		(dnp no)
 		(fields_autoplaced yes)
-		(property "Reference" "#PWR032"
+		(property "Reference" "#PWR038"
 			(at 260.35 86.36 0)
 			(effects
@@
 			(project "BQ76925_ATMEGA328P_6S_20A_BMS"
 				(path "/624a087f-322b-4a70-8c29-0e4f8f018e16/e88de734-726e-4991-811a-b88126c63525"
-					(reference "#PWR032")
+					(reference "#PWR038")
 					(unit 1)
 				)
@@
 		(dnp no)
 		(fields_autoplaced yes)
-		(property "Reference" "#PWR035"
+		(property "Reference" "#PWR037"
 			(at 256.54 142.24 0)
 			(effects
@@
 			(project "BQ76925_ATMEGA328P_6S_20A_BMS"
 				(path "/624a087f-322b-4a70-8c29-0e4f8f018e16/e88de734-726e-4991-811a-b88126c63525"
-					(reference "#PWR035")
+					(reference "#PWR037")
 					(unit 1)
 				)
@@
 		(dnp no)
 		(fields_autoplaced yes)
-		(property "Reference" "R27"
+		(property "Reference" "R28"
 			(at 262.89 67.3099 0)
 			(effects
@@
 			(project "BQ76925_ATMEGA328P_6S_20A_BMS"
 				(path "/624a087f-322b-4a70-8c29-0e4f8f018e16/e88de734-726e-4991-811a-b88126c63525"
-					(reference "R27")
+					(reference "R28")
 					(unit 1)
 				)
@@
 		(dnp no)
 		(fields_autoplaced yes)
-		(property "Reference" "C26"
+		(property "Reference" "C23"
 			(at 82.55 175.2662 0)
 			(effects
@@
 			(project "BQ76925_ATMEGA328P_6S_20A_BMS"
 				(path "/624a087f-322b-4a70-8c29-0e4f8f018e16/e88de734-726e-4991-811a-b88126c63525"
-					(reference "C26")
+					(reference "C23")
 					(unit 1)
 				)
@@
 		(dnp no)
 		(fields_autoplaced yes)
-		(property "Reference" "R28"
+		(property "Reference" "R27"
 			(at 259.08 118.1099 0)
 			(effects
@@
 			(project "BQ76925_ATMEGA328P_6S_20A_BMS"
 				(path "/624a087f-322b-4a70-8c29-0e4f8f018e16/e88de734-726e-4991-811a-b88126c63525"
-					(reference "R28")
+					(reference "R27")
 					(unit 1)
 				)
@@
 		(dnp no)
 		(fields_autoplaced yes)
-		(property "Reference" "#PWR037"
+		(property "Reference" "#PWR034"
 			(at 123.19 175.26 0)
 			(effects
@@
 			(project "BQ76925_ATMEGA328P_6S_20A_BMS"
 				(path "/624a087f-322b-4a70-8c29-0e4f8f018e16/e88de734-726e-4991-811a-b88126c63525"
-					(reference "#PWR037")
+					(reference "#PWR034")
 					(unit 1)
 				)
@@
 		(dnp no)
 		(fields_autoplaced yes)
-		(property "Reference" "#PWR033"
+		(property "Reference" "#PWR036"
 			(at 256.54 116.84 0)
 			(effects
@@
 			(project "BQ76925_ATMEGA328P_6S_20A_BMS"
 				(path "/624a087f-322b-4a70-8c29-0e4f8f018e16/e88de734-726e-4991-811a-b88126c63525"
-					(reference "#PWR033")
+					(reference "#PWR036")
 					(unit 1)
 				)
@@
 		(dnp no)
 		(fields_autoplaced yes)
-		(property "Reference" "#PWR038"
+		(property "Reference" "#PWR033"
 			(at 107.95 189.23 0)
 			(effects
@@
 			(project "BQ76925_ATMEGA328P_6S_20A_BMS"
 				(path "/624a087f-322b-4a70-8c29-0e4f8f018e16/e88de734-726e-4991-811a-b88126c63525"
-					(reference "#PWR038")
+					(reference "#PWR033")
 					(unit 1)
 				)
@@
 		(dnp no)
 		(fields_autoplaced yes)
-		(property "Reference" "J5"
+		(property "Reference" "J6"
 			(at 266.7 34.2899 0)
 			(effects
@@
 			(project "BQ76925_ATMEGA328P_6S_20A_BMS"
 				(path "/624a087f-322b-4a70-8c29-0e4f8f018e16/e88de734-726e-4991-811a-b88126c63525"
-					(reference "J5")
+					(reference "J6")
 					(unit 1)
 				)
@@
 		(dnp no)
 		(fields_autoplaced yes)
-		(property "Reference" "C28"
+		(property "Reference" "C21"
 			(at 67.31 175.2662 0)
 			(effects
@@
 			(project "BQ76925_ATMEGA328P_6S_20A_BMS"
 				(path "/624a087f-322b-4a70-8c29-0e4f8f018e16/e88de734-726e-4991-811a-b88126c63525"
-					(reference "C28")
+					(reference "C21")
 					(unit 1)
 				)
@@
 		(dnp no)
 		(fields_autoplaced yes)
-		(property "Reference" "C21"
+		(property "Reference" "C24"
 			(at 83.82 43.1862 0)
 			(effects
@@
 			(project "BQ76925_ATMEGA328P_6S_20A_BMS"
 				(path "/624a087f-322b-4a70-8c29-0e4f8f018e16/e88de734-726e-4991-811a-b88126c63525"
-					(reference "C21")
+					(reference "C24")
 					(unit 1)
 				)
@@
 		(dnp no)
 		(fields_autoplaced yes)
-		(property "Reference" "C20"
+		(property "Reference" "C22"
 			(at 72.39 42.7481 0)
 			(effects
@@
 			(project "BQ76925_ATMEGA328P_6S_20A_BMS"
 				(path "/624a087f-322b-4a70-8c29-0e4f8f018e16/e88de734-726e-4991-811a-b88126c63525"
-					(reference "C20")
+					(reference "C22")
 					(unit 1)
 				)
@@
 		(dnp no)
 		(fields_autoplaced yes)
-		(property "Reference" "#PWR036"
+		(property "Reference" "#PWR027"
 			(at 60.96 173.99 0)
 			(effects
@@
 			(project "BQ76925_ATMEGA328P_6S_20A_BMS"
 				(path "/624a087f-322b-4a70-8c29-0e4f8f018e16/e88de734-726e-4991-811a-b88126c63525"
-					(reference "#PWR036")
+					(reference "#PWR027")
 					(unit 1)
 				)
@@
 		(dnp no)
 		(fields_autoplaced yes)
-		(property "Reference" "C27"
+		(property "Reference" "C26"
 			(at 116.84 175.2662 0)
 			(effects
@@
 			(project "BQ76925_ATMEGA328P_6S_20A_BMS"
 				(path "/624a087f-322b-4a70-8c29-0e4f8f018e16/e88de734-726e-4991-811a-b88126c63525"
-					(reference "C27")
+					(reference "C26")
 					(unit 1)
 				)
@@
 		(dnp no)
 		(fields_autoplaced yes)
-		(property "Reference" "#PWR027"
+		(property "Reference" "#PWR030"
 			(at 86.36 36.83 0)
 			(effects
@@
 			(project "BQ76925_ATMEGA328P_6S_20A_BMS"
 				(path "/624a087f-322b-4a70-8c29-0e4f8f018e16/e88de734-726e-4991-811a-b88126c63525"
-					(reference "#PWR027")
+					(reference "#PWR030")
 					(unit 1)
 				)
@@
 		(dnp no)
 		(fields_autoplaced yes)
-		(property "Reference" "#PWR030"
+		(property "Reference" "#PWR032"
 			(at 100.33 55.88 0)
 			(effects
@@
 			(project "BQ76925_ATMEGA328P_6S_20A_BMS"
 				(path "/624a087f-322b-4a70-8c29-0e4f8f018e16/e88de734-726e-4991-811a-b88126c63525"
-					(reference "#PWR030")
+					(reference "#PWR032")
 					(unit 1)
 				)
@@
 		(dnp no)
 		(fields_autoplaced yes)
-		(property "Reference" "J6"
+		(property "Reference" "J5"
 			(at 204.47 119.38 0)
 			(effects
@@
 			(project "BQ76925_ATMEGA328P_6S_20A_BMS"
 				(path "/624a087f-322b-4a70-8c29-0e4f8f018e16/e88de734-726e-4991-811a-b88126c63525"
-					(reference "J6")
+					(reference "J5")
 					(unit 1)
 				)
@@
 		(dnp no)
 		(fields_autoplaced yes)
-		(property "Reference" "#PWR039"
+		(property "Reference" "#PWR035"
 			(at 203.2 60.96 0)
 			(effects
@@
 			(project "BQ76925_ATMEGA328P_6S_20A_BMS"
 				(path "/624a087f-322b-4a70-8c29-0e4f8f018e16/e88de734-726e-4991-811a-b88126c63525"
-					(reference "#PWR039")
+					(reference "#PWR035")
 					(unit 1)
 				)
@@
 		(on_board yes)
 		(dnp no)
-		(property "Reference" "Y2"
+		(property "Reference" "Y1"
 			(at 203.2 44.45 0)
 			(effects
@@
 			(project "BQ76925_ATMEGA328P_6S_20A_BMS"
 				(path "/624a087f-322b-4a70-8c29-0e4f8f018e16/e88de734-726e-4991-811a-b88126c63525"
-					(reference "Y2")
+					(reference "Y1")
 					(unit 1)
 				)
@@
 		(dnp no)
 		(fields_autoplaced yes)
-		(property "Reference" "C22"
+		(property "Reference" "C25"
 			(at 102.87 43.1862 0)
 			(effects
@@
 			(project "BQ76925_ATMEGA328P_6S_20A_BMS"
 				(path "/624a087f-322b-4a70-8c29-0e4f8f018e16/e88de734-726e-4991-811a-b88126c63525"
-					(reference "C22")
-					(unit 1)
-				)
+					(reference "C25")
+					(unit 1)
+				)

Commit message: pcb placement and 90 percent routed
Connections:
- net +5V: now also J5.2 (Pin_2); no longer J5.6 (Pin_6)
- net GND: now also J5.6 (Pin_6); no longer J5.4 (Pin_4)
- net MOSI: now also J5.4 (Pin_4); no longer J5.5 (Pin_5)
- net SCK: now also J5.3 (Pin_3); no longer J5.2 (Pin_2)
- net VCOUT: now also U3.25 (PC2); no longer U3.26 (PC3)
- net VIOUT: now also U3.26 (PC3); no longer U3.25 (PC2)
- net ~{RESET}: now also J5.5 (Pin_5); no longer J5.3 (Pin_3)
Changed lines of the file:
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@@
 	)
 	(label "5V"
-		(at 226.06 125.73 180)
-		(fields_autoplaced yes)
-		(effects
-			(font
-				(size 1.27 1.27)
-			)
-			(justify right bottom)
+		(at 182.88 128.27 0)
+		(fields_autoplaced yes)
+		(effects
+			(font
+				(size 1.27 1.27)
+			)
+			(justify left bottom)
 		)
 	)
@@
 	)
 	(label "GND"
-		(at 226.06 130.81 180)
+		(at 226.06 125.73 180)
 		(fields_autoplaced yes)
 		(effects
@@
 	)
 	(label "SCK"
-		(at 182.88 128.27 0)
+		(at 182.88 130.81 0)
 		(fields_autoplaced yes)
 		(effects
@@
 	)
 	(label "~{RESET}"
-		(at 182.88 130.81 0)
-		(fields_autoplaced yes)
-		(effects
-			(font
-				(size 1.27 1.27)
-			)
-			(justify left bottom)
+		(at 226.06 128.27 180)
+		(fields_autoplaced yes)
+		(effects
+			(font
+				(size 1.27 1.27)
+			)
+			(justify right bottom)
 		)
 	)
@@
 	)
 	(label "MOSI"
-		(at 226.06 128.27 180)
+		(at 226.06 130.81 180)
 		(fields_autoplaced yes)
 		(effects
@@
 	(hierarchical_label "VIOUT"
 		(shape input)
-		(at 123.19 88.9 0)
+		(at 123.19 91.44 0)
 		(fields_autoplaced yes)
 		(effects
@@
 	(hierarchical_label "VCOUT"
 		(shape input)
-		(at 123.19 91.44 0)
-		(fields_autoplaced yes)
-		(effects
+		(at 123.19 88.9 0)
+		(fields_autoplaced yes)
+		(effects
