File: electronics/PCB_BQ76925_ATMEGA328P_6S_20A_BMS/Atmega328P.kicad_sch (KiCad schematic)
At the start: 15 parts, among them J5 Conn_02x03, J6 Conn_01x04, U3 ATmega328P-A, U4 AMS1117-5.0, Y1 16Mhz

Commit message: PCB DRC complete footprints library exported. PCB optimization required
Parts:
- C21, C22, C26: footprint Capacitor_SMD:C_0603_1608Metric_Pad1.08x0.95mm_HandSolder -> BQ76925_ATMEGA328P_6S_20A_BMS:C_0603_1608Metric_Pad1.08x0.95mm_HandSolder
- C23, C24, C25, C27: footprint Capacitor_SMD:C_0805_2012Metric_Pad1.18x1.45mm_HandSolder -> BQ76925_ATMEGA328P_6S_20A_BMS:C_0805_2012Metric_Pad1.18x1.45mm_HandSolder
- D7: footprint Resistor_SMD:R_0805_2012Metric_Pad1.20x1.40mm_HandSolder -> BQ76925_ATMEGA328P_6S_20A_BMS:R_0805_2012Metric_Pad1.20x1.40mm_HandSolder
- J5: footprint Connector_PinHeader_2.54mm:PinHeader_2x03_P2.54mm_Vertical -> BQ76925_ATMEGA328P_6S_20A_BMS:PinHeader_2x03_P2.54mm_Vertical
- J6: footprint Connector_PinHeader_2.54mm:PinHeader_1x04_P2.54mm_Vertical -> BQ76925_ATMEGA328P_6S_20A_BMS:PinHeader_1x04_P2.54mm_Vertical
- R27, R28: footprint Resistor_SMD:R_0603_1608Metric_Pad0.98x0.95mm_HandSolder -> BQ76925_ATMEGA328P_6S_20A_BMS:R_0603_1608Metric_Pad0.98x0.95mm_HandSolder
- U3: footprint Package_QFP:TQFP-32_7x7mm_P0.8mm -> BQ76925_ATMEGA328P_6S_20A_BMS:TQFP-32_7x7mm_P0.8mm
- U4: footprint Package_TO_SOT_SMD:SOT-223-3_TabPin2 -> BQ76925_ATMEGA328P_6S_20A_BMS:SOT-223-3_TabPin2
- Y1: footprint Crystal:Resonator_SMD_Murata_CSTxExxV-3Pin_3.0x1.1mm_HandSoldering -> BQ76925_ATMEGA328P_6S_20A_BMS:Resonator_SMD_Murata_CSTxExxV-3Pin_3.0x1.1mm_HandSoldering
Connections:
- net MISO: now also R28.1
- net SCK: no longer R28.1
- net SW: now also U3.13 (PB1); no longer U3.1 (PD3)
Changed lines of the file:
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@@
 	)
 	(no_connect
-		(at 106.68 63.5)
+		(at 106.68 111.76)
 	)
 	(no_connect
@@
 	(wire
 		(pts
-			(xy 106.68 111.76) (xy 123.19 111.76)
+			(xy 106.68 63.5) (xy 123.19 63.5)
 		)
 		(stroke
@@
 		)
 	)
-	(label "SCK"
-		(at 255.27 63.5 0)
-		(fields_autoplaced yes)
-		(effects
-			(font
-				(size 1.27 1.27)
-			)
-			(justify left bottom)
-		)
-	)
 	(label "MOSI"
 		(at 121.92 68.58 180)
@@
 	(label "GND"
 		(at 243.84 39.37 0)
+		(fields_autoplaced yes)
+		(effects
+			(font
+				(size 1.27 1.27)
+			)
+			(justify left bottom)
+		)
+	)
+	(label "MISO"
+		(at 255.27 63.5 0)
 		(fields_autoplaced yes)
 		(effects
@@
 	(hierarchical_label "SW"
 		(shape output)
-		(at 123.19 111.76 0)
+		(at 123.19 63.5 0)
 		(fields_autoplaced yes)
 		(effects
@@
 			)
 		)
-		(property "Footprint" "Capacitor_SMD:C_0805_2012Metric_Pad1.18x1.45mm_HandSolder"
+		(property "Footprint" "BQ76925_ATMEGA328P_6S_20A_BMS:C_0805_2012Metric_Pad1.18x1.45mm_HandSolder"
 			(at 256.54 130.81 0)
 			(effects
@@
 			)
 		)
-		(property "Footprint" "Resistor_SMD:R_0603_1608Metric_Pad0.98x0.95mm_HandSolder"
+		(property "Footprint" "BQ76925_ATMEGA328P_6S_20A_BMS:R_0603_1608Metric_Pad0.98x0.95mm_HandSolder"
 			(at 260.35 68.58 0)
 			(effects
@@
 			)
 		)
-		(property "Footprint" "Capacitor_SMD:C_0805_2012Metric_Pad1.18x1.45mm_HandSolder"
+		(property "Footprint" "BQ76925_ATMEGA328P_6S_20A_BMS:C_0805_2012Metric_Pad1.18x1.45mm_HandSolder"
 			(at 80.01 176.53 0)
 			(effects
@@
 			)
 		)
-		(property "Footprint" "Resistor_SMD:R_0603_1608Metric_Pad0.98x0.95mm_HandSolder"
+		(property "Footprint" "BQ76925_ATMEGA328P_6S_20A_BMS:R_0603_1608Metric_Pad0.98x0.95mm_HandSolder"
 			(at 256.54 119.38 0)
 			(effects
@@
 			)
 		)
-		(property "Footprint" "Package_QFP:TQFP-32_7x7mm_P0.8mm"
+		(property "Footprint" "BQ76925_ATMEGA328P_6S_20A_BMS:TQFP-32_7x7mm_P0.8mm"
 			(at 91.44 91.44 0)
 			(effects
@@
 			)
 		)
-		(property "Footprint" "Connector_PinHeader_2.54mm:PinHeader_1x04_P2.54mm_Vertical"
+		(property "Footprint" "BQ76925_ATMEGA328P_6S_20A_BMS:PinHeader_1x04_P2.54mm_Vertical"
 			(at 264.16 34.29 0)
 			(effects
@@
 			)
 		)
-		(property "Footprint" "Capacitor_SMD:C_0603_1608Metric_Pad1.08x0.95mm_HandSolder"
+		(property "Footprint" "BQ76925_ATMEGA328P_6S_20A_BMS:C_0603_1608Metric_Pad1.08x0.95mm_HandSolder"
 			(at 64.77 176.53 0)
 			(effects
@@
 			)
 		)
-		(property "Footprint" "Capacitor_SMD:C_0805_2012Metric_Pad1.18x1.45mm_HandSolder"
+		(property "Footprint" "BQ76925_ATMEGA328P_6S_20A_BMS:C_0805_2012Metric_Pad1.18x1.45mm_HandSolder"
 			(at 81.28 44.45 0)
 			(effects
@@
 			)
 		)
-		(property "Footprint" "Capacitor_SMD:C_0603_1608Metric_Pad1.08x0.95mm_HandSolder"
+		(property "Footprint" "BQ76925_ATMEGA328P_6S_20A_BMS:C_0603_1608Metric_Pad1.08x0.95mm_HandSolder"
 			(at 69.85 44.45 0)
 			(effects
@@
 			)
 		)
-		(property "Footprint" "Capacitor_SMD:C_0603_1608Metric_Pad1.08x0.95mm_HandSolder"
+		(property "Footprint" "BQ76925_ATMEGA328P_6S_20A_BMS:C_0603_1608Metric_Pad1.08x0.95mm_HandSolder"
 			(at 114.3 176.53 0)
 			(effects
@@
 			)
 		)
-		(property "Footprint" "Package_TO_SOT_SMD:SOT-223-3_TabPin2"
+		(property "Footprint" "BQ76925_ATMEGA328P_6S_20A_BMS:SOT-223-3_TabPin2"
 			(at 101.6 167.64 0)
 			(effects
@@
 			)
 		)
-		(property "Footprint" "Resistor_SMD:R_0805_2012Metric_Pad1.20x1.40mm_HandSolder"
+		(property "Footprint" "BQ76925_ATMEGA328P_6S_20A_BMS:R_0805_2012Metric_Pad1.20x1.40mm_HandSolder"
 			(at 260.35 74.93 90)
 			(effects
@@
 			)
 		)
-		(property "Footprint" "Connector_PinHeader_2.54mm:PinHeader_2x03_P2.54mm_Vertical"
+		(property "Footprint" "BQ76925_ATMEGA328P_6S_20A_BMS:PinHeader_2x03_P2.54mm_Vertical"
 			(at 203.2 128.27 0)
 			(effects
@@
 			)
 		)
-		(property "Footprint" "Crystal:Resonator_SMD_Murata_CSTxExxV-3Pin_3.0x1.1mm_HandSoldering"
+		(property "Footprint" "BQ76925_ATMEGA328P_6S_20A_BMS:Resonator_SMD_Murata_CSTxExxV-3Pin_3.0x1.1mm_HandSoldering"
 			(at 203.2 50.8 0)
 			(effects
@@
 			)
 		)
-		(property "Footprint" "Capacitor_SMD:C_0805_2012Metric_Pad1.18x1.45mm_HandSolder"
+		(property "Footprint" "BQ76925_ATMEGA328P_6S_20A_BMS:C_0805_2012Metric_Pad1.18x1.45mm_HandSolder"
 			(at 100.33 44.45 0)
 			(effects
