File: electronics/PCB_BQ76925_ATMEGA328P_6S_20A_BMS/BQ76925_Schematic.kicad_sch (KiCad schematic)
At the start: 35 parts, among them J1 Conn_01x09, J3 Conn_01x02, U1 BQ76925PW

Commit message: schematic completed component need to be finalised
Parts:
- C23: footprint (none) -> Capacitor_SMD:C_1206_3216Metric_Pad1.33x1.80mm_HandSolder
Connections:
- net +BATT: now reaches D1.2 (A), J1.1 (Pin_1)
Other:
- note added: "BQ76925 Schematic 24V 6 Cell Monitoring"
- note added: "~{TVNBTEk=}"
- company: (none) -> M S Ali
- title: (none) -> Raven-I Sentinel
Changed lines of the file:
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@@
 	(generator_version "8.0")
 	(paper "A4")
+	(title_block
+		(title "Raven-I Sentinel")
+		(company "M S Ali")
+	)
 	(junction
 		(at 102.87 66.04)
@@
 	)
 	(junction
+		(at 62.23 78.74)
+		(diameter 0)
+		(color 0 0 0 0)
+	)
+	(junction
 		(at 144.78 144.78)
 		(diameter 0)
@@
 	(wire
 		(pts
+			(xy 62.23 76.2) (xy 62.23 78.74)
+		)
+		(stroke
+			(width 0)
+			(type default)
+		)
+	)
+	(wire
+		(pts
 			(xy 55.88 99.06) (xy 69.85 99.06)
 		)
@@
 	(wire
 		(pts
+			(xy 62.23 78.74) (xy 55.88 78.74)
+		)
+		(stroke
+			(width 0)
+			(type default)
+		)
+	)
+	(wire
+		(pts
 			(xy 213.36 78.74) (xy 217.17 78.74)
 		)
@@
 	(wire
 		(pts
-			(xy 71.12 78.74) (xy 55.88 78.74)
+			(xy 71.12 78.74) (xy 62.23 78.74)
 		)
 		(stroke
@@
 		)
 	)
+	(text "~{TVNBTEk=}"
+		(exclude_from_sim no)
+		(at 272.796 173.99 0)
+		(effects
+			(font
+				(face "Symbol")
+				(size 3 3)
+				(color 132 0 0 1)
+			)
+		)
+	)
+	(text "BQ76925 Schematic 24V 6 Cell Monitoring"
+		(exclude_from_sim no)
+		(at 63.5 20.828 0)
+		(effects
+			(font
+				(face "Times New Roman")
+				(size 3.81 3.81)
+			)
+		)
+	)
 	(hierarchical_label "PACK-"
 		(shape input)
@@
 	)
 	(symbol
+		(lib_id "BQ76925_ATMEGA328P_6S_20A_BMS:+BATT")
+		(at 62.23 76.2 0)
+		(unit 1)
+		(exclude_from_sim no)
+		(in_bom yes)
+		(on_board yes)
+		(dnp no)
+		(fields_autoplaced yes)
+		(property "Reference" "#PWR034"
+			(at 62.23 80.01 0)
+			(effects
+				(font
+					(size 1.27 1.27)
+				)
+				(hide yes)
+			)
+		)
+		(property "Value" "+BATT"
+			(at 62.23 71.12 0)
+			(effects
+				(font
+					(size 1.27 1.27)
+				)
+			)
+		)
+		(property "Footprint" ""
+			(at 62.23 76.2 0)
+			(effects
+				(font
+					(size 1.27 1.27)
+				)
+				(hide yes)
+			)
+		)
+		(property "Datasheet" ""
+			(at 62.23 76.2 0)
+			(effects
+				(font
+					(size 1.27 1.27)
+				)
+				(hide yes)
+			)
+		)
+		(property "Description" "Power symbol creates a global label with name \"+BATT\""
+			(at 62.23 76.2 0)
+			(effects
+				(font
+					(size 1.27 1.27)
+				)
+				(hide yes)
+			)
+		)
+		(pin "1"
+		)
+		(instances
+			(project "BQ76925_ATMEGA328P_6S_20A_BMS"
+				(path "/624a087f-322b-4a70-8c29-0e4f8f018e16/87862f27-26e3-4a63-80aa-70bc4698f5cc"
+					(reference "#PWR034")
+					(unit 1)
+				)
+			)
+		)
+	)
+	(symbol
 		(lib_id "BQ76925_ATMEGA328P_6S_20A_BMS:R_Small_US")
 		(at 240.03 73.66 180)
@@
 			)
 		)
-		(property "Footprint" ""
+		(property "Footprint" "Capacitor_SMD:C_1206_3216Metric_Pad1.33x1.80mm_HandSolder"
 			(at 264.16 95.25 0)
 			(effects

Commit message: Schematic completed components calculated need to check avaialability
Parts:
- C10: footprint (none) -> Capacitor_SMD:C_0603_1608Metric_Pad1.08x0.95mm_HandSolder
- C11: renamed from C16; footprint (none) -> Capacitor_SMD:C_0805_2012Metric_Pad1.18x1.45mm_HandSolder
- C12: renamed from C17; footprint (none) -> Capacitor_SMD:C_0805_2012Metric_Pad1.18x1.45mm_HandSolder
- C13: renamed from C11; footprint (none) -> Capacitor_SMD:C_0603_1608Metric_Pad1.08x0.95mm_HandSolder
- C14: renamed from C18; footprint (none) -> Capacitor_SMD:C_0805_2012Metric_Pad1.18x1.45mm_HandSolder
- C2: renamed from C12; footprint (none) -> Capacitor_SMD:C_0805_2012Metric_Pad1.18x1.45mm_HandSolder
- C4: renamed from C13; footprint (none) -> Capacitor_SMD:C_0805_2012Metric_Pad1.18x1.45mm_HandSolder
- C5: renamed from C14; footprint (none) -> Capacitor_SMD:C_0805_2012Metric_Pad1.18x1.45mm_HandSolder
- C6: renamed from C15; footprint (none) -> Capacitor_SMD:C_0805_2012Metric_Pad1.18x1.45mm_HandSolder
- C7: renamed from C24; footprint (none) -> Capacitor_SMD:C_0805_2012Metric_Pad1.18x1.45mm_HandSolder
- C8: renamed from C22; footprint (none) -> Capacitor_SMD:C_0603_1608Metric_Pad1.08x0.95mm_HandSolder
- D2: value BZT52C30-13-F -> 30V
- R9: renamed from R10; footprint (none) -> Resistor_SMD:R_0603_1608Metric_Pad0.98x0.95mm_HandSolder
- renumbered C19 to C1, C20 to C3, C23 to C9, J1 to J3, J3 to J4, R9 to R1, R19 to R10, R20 to R11, R21 to R12, R11 to R13, R12 to R14, R13 to R15, R14 to R16, R15 to R2, R16 to R3, R23 to R4, R22 to R5, R24 to R6, R17 to R7, R18 to R8

Commit message: common footprints assigned to symbols
Parts:
- C1: value 10uF/50V -> 22uF/35V; footprint (none) -> Capacitor_SMD:CP_Elec_6.3x5.7
- C10, C13, C8: value 0.1uF -> 100nF/50V; footprint Capacitor_SMD:C_0603_1608Metric_Pad1.08x0.95mm_HandSolder -> Capacitor_SMD:C_0805_2012Metric_Pad1.18x1.45mm_HandSolder
- C11, C12, C14, C2, C4, C5, C6, C7: value 1uF -> 1uF/50V
- C3: value 4.7uF/10V -> 4.7uF/25V; footprint (none) -> Capacitor_SMD:C_0805_2012Metric_Pad1.18x1.45mm_HandSolder
- R1, R10, R11, R12, R2, R3, R7, R8: footprint (none) -> Resistor_SMD:R_1206_3216Metric_Pad1.30x1.75mm_HandSolder
- R13, R14, R4, R5, R6: footprint (none) -> Resistor_SMD:R_0603_1608Metric_Pad0.98x0.95mm_HandSolder
Changed lines of the file:
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@@
 			)
 		)
-		(property "Footprint" ""
+		(property "Footprint" "Resistor_SMD:R_1206_3216Metric_Pad1.30x1.75mm_HandSolder"
 			(at 90.17 123.19 0)
 			(effects
@@
 			)
 		)
-		(property "Footprint" ""
+		(property "Footprint" "Resistor_SMD:R_0603_1608Metric_Pad0.98x0.95mm_HandSolder"
 			(at 213.36 73.66 0)
 			(effects
@@
 			)
 		)
-		(property "Value" "4.7uF/10V"
+		(property "Value" "4.7uF/25V"
 			(at 154.94 69.8562 0)
 			(effects
@@
 			)
 		)
-		(property "Footprint" ""
+		(property "Footprint" "Capacitor_SMD:C_0805_2012Metric_Pad1.18x1.45mm_HandSolder"
 			(at 152.4 68.58 0)
 			(effects
@@
 			)
 		)
-		(property "Footprint" ""
+		(property "Footprint" "Resistor_SMD:R_0603_1608Metric_Pad0.98x0.95mm_HandSolder"
 			(at 240.03 73.66 0)
 			(effects
@@
 			)
 		)
-		(property "Footprint" ""
+		(property "Footprint" "Resistor_SMD:R_1206_3216Metric_Pad1.30x1.75mm_HandSolder"
 			(at 90.17 100.33 0)
 			(effects
@@
 			)
 		)
-		(property "Footprint" ""
+		(property "Footprint" "Resistor_SMD:R_1206_3216Metric_Pad1.30x1.75mm_HandSolder"
 			(at 90.17 111.76 0)
 			(effects
@@
 			)
 		)
-		(property "Value" "1uF"
+		(property "Value" "1uF/50V"
 			(at 105.41 82.5562 0)
 			(effects
@@
 			)
 		)
-		(property "Value" "1uF"
+		(property "Value" "1uF/50V"
 			(at 105.41 105.4162 0)
 			(effects
@@
 			)
 		)
-		(property "Footprint" ""
+		(property "Footprint" "Resistor_SMD:R_1206_3216Metric_Pad1.30x1.75mm_HandSolder"
 			(at 90.17 88.9 0)
 			(effects
@@
 			)
 		)
-		(property "Footprint" ""
+		(property "Footprint" "Resistor_SMD:R_1206_3216Metric_Pad1.30x1.75mm_HandSolder"
 			(at 90.17 77.47 0)
 			(effects
@@
 			)
 		)
-		(property "Footprint" ""
+		(property "Footprint" "Resistor_SMD:R_0603_1608Metric_Pad0.98x0.95mm_HandSolder"
 			(at 264.16 73.66 0)
 			(effects
@@
 			)
 		)
-		(property "Value" "0.1uF"
+		(property "Value" "100nF/50V"
 			(at 242.57 96.5135 0)
 			(effects
@@
 			)
 		)
-		(property "Footprint" "Capacitor_SMD:C_0603_1608Metric_Pad1.08x0.95mm_HandSolder"
+		(property "Footprint" "Capacitor_SMD:C_0805_2012Metric_Pad1.18x1.45mm_HandSolder"
 			(at 240.03 95.25 0)
 			(effects
@@
 			)
 		)
-		(property "Footprint" ""
+		(property "Footprint" "Resistor_SMD:R_1206_3216Metric_Pad1.30x1.75mm_HandSolder"
 			(at 90.17 54.61 0)
 			(effects
@@
 			)
 		)
-		(property "Footprint" ""
+		(property "Footprint" "Resistor_SMD:R_0603_1608Metric_Pad0.98x0.95mm_HandSolder"
 			(at 144.78 129.54 0)
 			(effects
@@
 			)
 		)
-		(property "Value" "1uF"
+		(property "Value" "1uF/50V"
 			(at 105.41 128.2762 0)
 			(effects
@@
 			)
 		)
-		(property "Value" "1uF"
+		(property "Value" "1uF/50V"
 			(at 105.41 59.6962 0)
 			(effects
@@
 			)
 		)
-		(property "Value" "1uF"
+		(property "Value" "1uF/50V"
 			(at 105.41 71.1262 0)
 			(effects
@@
 			)
 		)
-		(property "Footprint" ""
+		(property "Footprint" "Resistor_SMD:R_1206_3216Metric_Pad1.30x1.75mm_HandSolder"
 			(at 87.63 38.1 0)
 			(effects
@@
 			)
 		)
-		(property "Footprint" ""
+		(property "Footprint" "Resistor_SMD:R_0603_1608Metric_Pad0.98x0.95mm_HandSolder"
 			(at 176.53 129.54 0)
 			(effects
@@
 			)
 		)
-		(property "Value" "1uF"
+		(property "Value" "1uF/50V"
 			(at 215.9 96.5262 0)
 			(effects
@@
 			)
 		)
-		(property "Value" "0.1uF"
+		(property "Value" "100nF/50V"
 			(at 171.45 101.5935 0)
 			(effects
@@
 			)
 		)
-		(property "Footprint" "Capacitor_SMD:C_0603_1608Metric_Pad1.08x0.95mm_HandSolder"
+		(property "Footprint" "Capacitor_SMD:C_0805_2012Metric_Pad1.18x1.45mm_HandSolder"
 			(at 173.99 100.33 0)
 			(effects
@@
 			)
 		)
-		(property "Value" "1uF"
+		(property "Value" "1uF/50V"
 			(at 105.41 93.9862 0)
 			(effects
@@
 			)
 		)
-		(property "Value" "10uF/50V"
+		(property "Value" "22uF/35V"
 			(at 107.95 44.4562 0)
 			(effects
@@
 			)
 		)
-		(property "Footprint" ""
+		(property "Footprint" "Capacitor_SMD:CP_Elec_6.3x5.7"
 			(at 105.41 43.18 0)
 			(effects
@@
 			)
 		)
-		(property "Value" "0.1uF"
+		(property "Value" "100nF/50V"
 			(at 161.2963 118.11 90)
 			(effects
@@
 			)
 		)
-		(property "Footprint" "Capacitor_SMD:C_0603_1608Metric_Pad1.08x0.95mm_HandSolder"
+		(property "Footprint" "Capacitor_SMD:C_0805_2012Metric_Pad1.18x1.45mm_HandSolder"
 			(at 161.29 121.92 0)
 			(effects
@@
 			)
 		)
-		(property "Footprint" ""
+		(property "Footprint" "Resistor_SMD:R_1206_3216Metric_Pad1.30x1.75mm_HandSolder"
 			(at 90.17 66.04 0)
 			(effects
@@
 			)
 		)
-		(property "Value" "1uF"
+		(property "Value" "1uF/50V"
 			(at 105.41 116.8462 0)
 			(effects

Commit message: schematic components footprint updated
Parts:
- added D2: 40V, Diode_SMD:D_SMA_Handsoldering, symbol BQ76925_ATMEGA328P_6S_20A_BMS:D_TVS_Small_Filled
- D1: value MBR0540T1G -> SS24; footprint (none) -> Diode_SMD:D_SMB
- D3: renamed from D2; footprint (none) -> Diode_SMD:D_SOD-123
- J3: footprint (none) -> Connector_PinHeader_2.54mm:PinHeader_1x09_P2.54mm_Vertical
- J4: footprint (none) -> Connector_PinHeader_2.54mm:PinHeader_1x02_P2.54mm_Vertical
- R15, R16: footprint (none) -> Resistor_SMD:R_2512_6332Metric
Connections:
- net +BATT: now also D2.2 (A2)
- net GND: now also D2.1 (A1)
Other:
- moved on the sheet: D1, R1

Commit message: pcb design half complete
Parts:
- renumbered C2 to C1, C13 to C10, C10 to C11, C7 to C12, C8 to C13, C9 to C14, C4 to C2, C5 to C3, C6 to C4, C11 to C5, C12 to C6, C14 to C7, C1 to C8, C3 to C9, D2 to D1, D1 to D2, R2 to R1, R15 to R10, R16 to R11, R14 to R12, R9 to R13, R4 to R14, R5 to R15, R6 to R16, R3 to R2, R7 to R3, R8 to R4, R10 to R5, R11 to R6, R12 to R7, R1 to R8, R13 to R9

Commit message: routing issue analog pins parallel routing and more length need to plan
Connections:
- net A+: now reaches C10.1, R9.2, U1.11 (SENSEN)
- net A-: now reaches C10.2, R12.2, U1.12 (SENSEP)
Other:
- moved on the sheet: R12, R9
Changed lines of the file:
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@@
 	(wire
 		(pts
-			(xy 144.78 132.08) (xy 144.78 144.78)
+			(xy 144.78 137.16) (xy 144.78 144.78)
 		)
 		(stroke
@@
 	(wire
 		(pts
-			(xy 176.53 132.08) (xy 176.53 144.78)
+			(xy 176.53 137.16) (xy 176.53 144.78)
 		)
 		(stroke
@@
 	(wire
 		(pts
-			(xy 176.53 121.92) (xy 176.53 127)
+			(xy 176.53 121.92) (xy 176.53 132.08)
 		)
 		(stroke
@@
 	(wire
 		(pts
-			(xy 144.78 121.92) (xy 144.78 127)
+			(xy 144.78 121.92) (xy 144.78 132.08)
 		)
 		(stroke
@@
 		)
 	)
+	(label "A-"
+		(at 176.53 128.27 0)
+		(fields_autoplaced yes)
+		(effects
+			(font
+				(size 1.27 1.27)
+			)
+			(justify left bottom)
+		)
+	)
+	(label "A+"
+		(at 144.78 129.54 0)
+		(fields_autoplaced yes)
+		(effects
+			(font
+				(size 1.27 1.27)
+			)
+			(justify left bottom)
+		)
+	)
 	(hierarchical_label "PACK-"
 		(shape input)
@@
 	(symbol
 		(lib_id "BQ76925_ATMEGA328P_6S_20A_BMS:R_Small_US")
-		(at 144.78 129.54 180)
+		(at 144.78 134.62 180)
 		(unit 1)
 		(exclude_from_sim no)
@@
 		(fields_autoplaced yes)
 		(property "Reference" "R9"
-			(at 147.32 128.2699 0)
+			(at 147.32 133.3499 0)
 			(effects
 				(font
@@
 		)
 		(property "Value" "1k"
-			(at 147.32 130.8099 0)
+			(at 147.32 135.8899 0)
 			(effects
 				(font
@@
 		)
 		(property "Footprint" "Resistor_SMD:R_0603_1608Metric_Pad0.98x0.95mm_HandSolder"
-			(at 144.78 129.54 0)
+			(at 144.78 134.62 0)
 			(effects
 				(font
@@
 		)
 		(property "Datasheet" "~"
-			(at 144.78 129.54 0)
+			(at 144.78 134.62 0)
 			(effects
 				(font
@@
 		)
 		(property "Description" "Resistor, small US symbol"
-			(at 144.78 129.54 0)
+			(at 144.78 134.62 0)
 			(effects
 				(font
@@
 	(symbol
 		(lib_id "BQ76925_ATMEGA328P_6S_20A_BMS:R_Small_US")
-		(at 176.53 129.54 180)
+		(at 176.53 134.62 180)
 		(unit 1)
 		(exclude_from_sim no)
@@
 		(fields_autoplaced yes)
 		(property "Reference" "R12"
-			(at 179.07 128.2699 0)
+			(at 179.07 133.3499 0)
 			(effects
 				(font
@@
 		)
 		(property "Value" "1k"
-			(at 179.07 130.8099 0)
+			(at 179.07 135.8899 0)
 			(effects
 				(font
@@
 		)
 		(property "Footprint" "Resistor_SMD:R_0603_1608Metric_Pad0.98x0.95mm_HandSolder"
-			(at 176.53 129.54 0)
+			(at 176.53 134.62 0)
 			(effects
 				(font
@@
 		)
 		(property "Datasheet" "~"
-			(at 176.53 129.54 0)
+			(at 176.53 134.62 0)
 			(effects
 				(font
@@
 		)
 		(property "Description" "Resistor, small US symbol"
-			(at 176.53 129.54 0)
+			(at 176.53 134.62 0)
 			(effects
 				(font

Commit message: PCB DRC complete footprints library exported. PCB optimization required
Parts:
- C1, C10, C11, C12, C13, C2, C3, C4, C5, C6, C7, C9: footprint Capacitor_SMD:C_0805_2012Metric_Pad1.18x1.45mm_HandSolder -> BQ76925_ATMEGA328P_6S_20A_BMS:C_0805_2012Metric_Pad1.18x1.45mm_HandSolder
- C14: footprint Capacitor_SMD:C_1206_3216Metric_Pad1.33x1.80mm_HandSolder -> BQ76925_ATMEGA328P_6S_20A_BMS:C_1206_3216Metric_Pad1.33x1.80mm_HandSolder
- C8: footprint Capacitor_SMD:CP_Elec_6.3x5.7 -> BQ76925_ATMEGA328P_6S_20A_BMS:CP_Elec_6.3x5.7
- D1: footprint Diode_SMD:D_SMA_Handsoldering -> BQ76925_ATMEGA328P_6S_20A_BMS:D_SMA_Handsoldering
- D2: footprint Diode_SMD:D_SMB -> BQ76925_ATMEGA328P_6S_20A_BMS:D_SMB
- D3: footprint Diode_SMD:D_SOD-123 -> BQ76925_ATMEGA328P_6S_20A_BMS:D_SOD-123
- J3: footprint Connector_PinHeader_2.54mm:PinHeader_1x09_P2.54mm_Vertical -> BQ76925_ATMEGA328P_6S_20A_BMS:PinHeader_1x09_P2.54mm_Vertical
- J4: footprint Connector_PinHeader_2.54mm:PinHeader_1x02_P2.54mm_Vertical -> BQ76925_ATMEGA328P_6S_20A_BMS:PinHeader_1x02_P2.54mm_Vertical
- R1, R2, R3, R4, R5, R6, R7, R8: footprint Resistor_SMD:R_1206_3216Metric_Pad1.30x1.75mm_HandSolder -> BQ76925_ATMEGA328P_6S_20A_BMS:R_1206_3216Metric_Pad1.30x1.75mm_HandSolder
- R10, R11: footprint Resistor_SMD:R_2512_6332Metric -> BQ76925_ATMEGA328P_6S_20A_BMS:R_2512_6332Metric
- R12, R13, R14, R15, R16, R9: footprint Resistor_SMD:R_0603_1608Metric_Pad0.98x0.95mm_HandSolder -> BQ76925_ATMEGA328P_6S_20A_BMS:R_0603_1608Metric_Pad0.98x0.95mm_HandSolder
- U1: footprint Package_SO:TSSOP-20_4.4x6.5mm_P0.65mm -> BQ76925_ATMEGA328P_6S_20A_BMS:TSSOP-20_4.4x6.5mm_P0.65mm
Changed lines of the file:
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@@
 			)
 		)
-		(property "Footprint" "Resistor_SMD:R_1206_3216Metric_Pad1.30x1.75mm_HandSolder"
+		(property "Footprint" "BQ76925_ATMEGA328P_6S_20A_BMS:R_1206_3216Metric_Pad1.30x1.75mm_HandSolder"
 			(at 90.17 123.19 0)
 			(effects
@@
 			)
 		)
-		(property "Footprint" "Resistor_SMD:R_0603_1608Metric_Pad0.98x0.95mm_HandSolder"
+		(property "Footprint" "BQ76925_ATMEGA328P_6S_20A_BMS:R_0603_1608Metric_Pad0.98x0.95mm_HandSolder"
 			(at 213.36 73.66 0)
 			(effects
@@
 			)
 		)
-		(property "Footprint" "Capacitor_SMD:C_0805_2012Metric_Pad1.18x1.45mm_HandSolder"
+		(property "Footprint" "BQ76925_ATMEGA328P_6S_20A_BMS:C_0805_2012Metric_Pad1.18x1.45mm_HandSolder"
 			(at 152.4 68.58 0)
 			(effects
@@
 			)
 		)
-		(property "Footprint" "Resistor_SMD:R_0603_1608Metric_Pad0.98x0.95mm_HandSolder"
+		(property "Footprint" "BQ76925_ATMEGA328P_6S_20A_BMS:R_0603_1608Metric_Pad0.98x0.95mm_HandSolder"
 			(at 240.03 73.66 0)
 			(effects
@@
 			)
 		)
-		(property "Footprint" "Resistor_SMD:R_1206_3216Metric_Pad1.30x1.75mm_HandSolder"
+		(property "Footprint" "BQ76925_ATMEGA328P_6S_20A_BMS:R_1206_3216Metric_Pad1.30x1.75mm_HandSolder"
 			(at 90.17 100.33 0)
 			(effects
@@
 			)
 		)
-		(property "Footprint" "Resistor_SMD:R_1206_3216Metric_Pad1.30x1.75mm_HandSolder"
+		(property "Footprint" "BQ76925_ATMEGA328P_6S_20A_BMS:R_1206_3216Metric_Pad1.30x1.75mm_HandSolder"
 			(at 90.17 111.76 0)
 			(effects
@@
 			)
 		)
-		(property "Footprint" "Resistor_SMD:R_2512_6332Metric"
+		(property "Footprint" "BQ76925_ATMEGA328P_6S_20A_BMS:R_2512_6332Metric"
 			(at 161.544 138.684 90)
 			(effects
@@
 			)
 		)
-		(property "Footprint" "Capacitor_SMD:C_0805_2012Metric_Pad1.18x1.45mm_HandSolder"
+		(property "Footprint" "BQ76925_ATMEGA328P_6S_20A_BMS:C_0805_2012Metric_Pad1.18x1.45mm_HandSolder"
 			(at 102.87 81.28 0)
 			(effects
@@
 			)
 		)
-		(property "Footprint" "Capacitor_SMD:C_0805_2012Metric_Pad1.18x1.45mm_HandSolder"
+		(property "Footprint" "BQ76925_ATMEGA328P_6S_20A_BMS:C_0805_2012Metric_Pad1.18x1.45mm_HandSolder"
 			(at 102.87 104.14 0)
 			(effects
@@
 			)
 		)
-		(property "Footprint" "Resistor_SMD:R_1206_3216Metric_Pad1.30x1.75mm_HandSolder"
+		(property "Footprint" "BQ76925_ATMEGA328P_6S_20A_BMS:R_1206_3216Metric_Pad1.30x1.75mm_HandSolder"
 			(at 90.17 88.9 0)
 			(effects
@@
 			)
 		)
-		(property "Footprint" "Resistor_SMD:R_1206_3216Metric_Pad1.30x1.75mm_HandSolder"
+		(property "Footprint" "BQ76925_ATMEGA328P_6S_20A_BMS:R_1206_3216Metric_Pad1.30x1.75mm_HandSolder"
 			(at 90.17 77.47 0)
 			(effects
@@
 			)
 		)
-		(property "Footprint" "Resistor_SMD:R_0603_1608Metric_Pad0.98x0.95mm_HandSolder"
+		(property "Footprint" "BQ76925_ATMEGA328P_6S_20A_BMS:R_0603_1608Metric_Pad0.98x0.95mm_HandSolder"
 			(at 264.16 73.66 0)
 			(effects
@@
 			)
 		)
-		(property "Footprint" "Capacitor_SMD:C_0805_2012Metric_Pad1.18x1.45mm_HandSolder"
+		(property "Footprint" "BQ76925_ATMEGA328P_6S_20A_BMS:C_0805_2012Metric_Pad1.18x1.45mm_HandSolder"
 			(at 240.03 95.25 0)
 			(effects
@@
 			)
 		)
-		(property "Footprint" "Connector_PinHeader_2.54mm:PinHeader_1x02_P2.54mm_Vertical"
+		(property "Footprint" "BQ76925_ATMEGA328P_6S_20A_BMS:PinHeader_1x02_P2.54mm_Vertical"
 			(at 184.15 99.06 0)
 			(effects
@@
 			)
 		)
-		(property "Footprint" "Resistor_SMD:R_1206_3216Metric_Pad1.30x1.75mm_HandSolder"
+		(property "Footprint" "BQ76925_ATMEGA328P_6S_20A_BMS:R_1206_3216Metric_Pad1.30x1.75mm_HandSolder"
 			(at 90.17 54.61 0)
 			(effects
@@
 			)
 		)
-		(property "Footprint" "Resistor_SMD:R_0603_1608Metric_Pad0.98x0.95mm_HandSolder"
+		(property "Footprint" "BQ76925_ATMEGA328P_6S_20A_BMS:R_0603_1608Metric_Pad0.98x0.95mm_HandSolder"
 			(at 144.78 134.62 0)
 			(effects
@@
 			)
 		)
-		(property "Footprint" "Diode_SMD:D_SMA_Handsoldering"
+		(property "Footprint" "BQ76925_ATMEGA328P_6S_20A_BMS:D_SMA_Handsoldering"
 			(at 76.2 43.18 0)
 			(effects
@@
 			)
 		)
-		(property "Footprint" "Capacitor_SMD:C_0805_2012Metric_Pad1.18x1.45mm_HandSolder"
+		(property "Footprint" "BQ76925_ATMEGA328P_6S_20A_BMS:C_0805_2012Metric_Pad1.18x1.45mm_HandSolder"
 			(at 102.87 127 0)
 			(effects
@@
 			)
 		)
-		(property "Footprint" "Capacitor_SMD:C_0805_2012Metric_Pad1.18x1.45mm_HandSolder"
+		(property "Footprint" "BQ76925_ATMEGA328P_6S_20A_BMS:C_0805_2012Metric_Pad1.18x1.45mm_HandSolder"
 			(at 102.87 58.42 0)
 			(effects
@@
 			)
 		)
-		(property "Footprint" "Capacitor_SMD:C_0805_2012Metric_Pad1.18x1.45mm_HandSolder"
+		(property "Footprint" "BQ76925_ATMEGA328P_6S_20A_BMS:C_0805_2012Metric_Pad1.18x1.45mm_HandSolder"
 			(at 102.87 69.85 0)
 			(effects
@@
 			)
 		)
-		(property "Footprint" "Resistor_SMD:R_1206_3216Metric_Pad1.30x1.75mm_HandSolder"
+		(property "Footprint" "BQ76925_ATMEGA328P_6S_20A_BMS:R_1206_3216Metric_Pad1.30x1.75mm_HandSolder"
 			(at 91.44 38.1 0)
 			(effects
@@
 			)
 		)
-		(property "Footprint" "Resistor_SMD:R_0603_1608Metric_Pad0.98x0.95mm_HandSolder"
+		(property "Footprint" "BQ76925_ATMEGA328P_6S_20A_BMS:R_0603_1608Metric_Pad0.98x0.95mm_HandSolder"
 			(at 176.53 134.62 0)
 			(effects
@@
 			)
 		)
-		(property "Footprint" "Capacitor_SMD:C_0805_2012Metric_Pad1.18x1.45mm_HandSolder"
+		(property "Footprint" "BQ76925_ATMEGA328P_6S_20A_BMS:C_0805_2012Metric_Pad1.18x1.45mm_HandSolder"
 			(at 213.36 95.25 0)
 			(effects
@@
 			)
 		)
-		(property "Footprint" "Connector_PinHeader_2.54mm:PinHeader_1x09_P2.54mm_Vertical"
+		(property "Footprint" "BQ76925_ATMEGA328P_6S_20A_BMS:PinHeader_1x09_P2.54mm_Vertical"
 			(at 50.8 88.9 0)
 			(effects
@@
 			)
 		)
-		(property "Footprint" "Package_SO:TSSOP-20_4.4x6.5mm_P0.65mm"
+		(property "Footprint" "BQ76925_ATMEGA328P_6S_20A_BMS:TSSOP-20_4.4x6.5mm_P0.65mm"
 			(at 135.636 102.87 0)
 			(effects
@@
 			)
 		)
-		(property "Footprint" "Diode_SMD:D_SOD-123"
+		(property "Footprint" "BQ76925_ATMEGA328P_6S_20A_BMS:D_SOD-123"
 			(at 97.79 43.18 90)
 			(effects
@@
 			)
 		)
-		(property "Footprint" "Capacitor_SMD:C_1206_3216Metric_Pad1.33x1.80mm_HandSolder"
+		(property "Footprint" "BQ76925_ATMEGA328P_6S_20A_BMS:C_1206_3216Metric_Pad1.33x1.80mm_HandSolder"
 			(at 264.16 95.25 0)
 			(effects
@@
 			)
 		)
-		(property "Footprint" "Resistor_SMD:R_0603_1608Metric_Pad0.98x0.95mm_HandSolder"
+		(property "Footprint" "BQ76925_ATMEGA328P_6S_20A_BMS:R_0603_1608Metric_Pad0.98x0.95mm_HandSolder"
 			(at 179.07 90.17 0)
 			(effects
@@
 			)
 		)
-		(property "Footprint" "Capacitor_SMD:C_0805_2012Metric_Pad1.18x1.45mm_HandSolder"
+		(property "Footprint" "BQ76925_ATMEGA328P_6S_20A_BMS:C_0805_2012Metric_Pad1.18x1.45mm_HandSolder"
 			(at 173.99 100.33 0)
 			(effects
@@
 			)
 		)
-		(property "Footprint" "Resistor_SMD:R_2512_6332Metric"
+		(property "Footprint" "BQ76925_ATMEGA328P_6S_20A_BMS:R_2512_6332Metric"
 			(at 161.544 148.844 90)
 			(effects
@@
 			)
 		)
-		(property "Footprint" "Capacitor_SMD:C_0805_2012Metric_Pad1.18x1.45mm_HandSolder"
+		(property "Footprint" "BQ76925_ATMEGA328P_6S_20A_BMS:C_0805_2012Metric_Pad1.18x1.45mm_HandSolder"
 			(at 102.87 92.71 0)
 			(effects
@@
 			)
 		)
-		(property "Footprint" "Capacitor_SMD:CP_Elec_6.3x5.7"
+		(property "Footprint" "BQ76925_ATMEGA328P_6S_20A_BMS:CP_Elec_6.3x5.7"
 			(at 105.41 43.18 0)
 			(effects
@@
 			)
 		)
-		(property "Footprint" "Capacitor_SMD:C_0805_2012Metric_Pad1.18x1.45mm_HandSolder"
+		(property "Footprint" "BQ76925_ATMEGA328P_6S_20A_BMS:C_0805_2012Metric_Pad1.18x1.45mm_HandSolder"
 			(at 161.29 121.92 0)
 			(effects
@@
 			)
 		)
-		(property "Footprint" "Resistor_SMD:R_1206_3216Metric_Pad1.30x1.75mm_HandSolder"
+		(property "Footprint" "BQ76925_ATMEGA328P_6S_20A_BMS:R_1206_3216Metric_Pad1.30x1.75mm_HandSolder"
 			(at 90.17 66.04 0)
 			(effects
@@
 			)
 		)
-		(property "Footprint" "Diode_SMD:D_SMB"
+		(property "Footprint" "BQ76925_ATMEGA328P_6S_20A_BMS:D_SMB"
 			(at 82.55 38.1 90)
 			(effects
@@
 			)
 		)
-		(property "Footprint" "Capacitor_SMD:C_0805_2012Metric_Pad1.18x1.45mm_HandSolder"
+		(property "Footprint" "BQ76925_ATMEGA328P_6S_20A_BMS:C_0805_2012Metric_Pad1.18x1.45mm_HandSolder"
 			(at 102.87 115.57 0)
 			(effects
